File: monitor-board/monitor-board.sch (KiCad schematic (older format))
At the start: 26 parts, among them J1 Conn_01x06, SW1 SW_IO12, SW2 SW_IO13, SW3 SW_IO14, SW4 SW_IO15, SW5 SW_IO32, SW6 SW_IO33, SW7 SW_IO34, SW8 SW_IO35, U1 ESP32-WROOM-32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

Commit message: Update footprints of resistors and led to go with cheap parts
Parts:
- D1: footprint LED_SMD:LED_0805_2012Metric_Pad1.15x1.40mm_HandSolder -> LED_SMD:LED_0603_1608Metric_Pad1.05x0.95mm_HandSolder
- R1, R10, R11, R2, R3, R4, R5, R6, R7, R8, R9: footprint Resistor_SMD:R_0805_2012Metric_Pad1.15x1.40mm_HandSolder -> Resistor_SMD:R_0603_1608Metric_Pad1.05x0.95mm_HandSolder
Changed lines of the file:
@@
 F 0 "R1" H 6320 2846 50  0000 L CNN
 F 1 "10k" H 6320 2755 50  0000 L CNN
-F 2 "Resistor_SMD:R_0805_2012Metric_Pad1.15x1.40mm_HandSolder" V 6180 2800 50  0001 C CNN
+F 2 "Resistor_SMD:R_0603_1608Metric_Pad1.05x0.95mm_HandSolder" V 6180 2800 50  0001 C CNN
 F 3 "~" H 6250 2800 50  0001 C CNN
 	1    6250 2800
@@
 F 0 "R2" H 6320 3496 50  0000 L CNN
 F 1 "10k" H 6320 3405 50  0000 L CNN
-F 2 "Resistor_SMD:R_0805_2012Metric_Pad1.15x1.40mm_HandSolder" V 6180 3450 50  0001 C CNN
+F 2 "Resistor_SMD:R_0603_1608Metric_Pad1.05x0.95mm_HandSolder" V 6180 3450 50  0001 C CNN
 F 3 "~" H 6250 3450 50  0001 C CNN
 	1    6250 3450
@@
 F 0 "R3" H 6320 4196 50  0000 L CNN
 F 1 "10k" H 6320 4105 50  0000 L CNN
-F 2 "Resistor_SMD:R_0805_2012Metric_Pad1.15x1.40mm_HandSolder" V 6180 4150 50  0001 C CNN
+F 2 "Resistor_SMD:R_0603_1608Metric_Pad1.05x0.95mm_HandSolder" V 6180 4150 50  0001 C CNN
 F 3 "~" H 6250 4150 50  0001 C CNN
 	1    6250 4150
@@
 F 0 "R4" H 6320 4846 50  0000 L CNN
 F 1 "10k" H 6320 4755 50  0000 L CNN
-F 2 "Resistor_SMD:R_0805_2012Metric_Pad1.15x1.40mm_HandSolder" V 6180 4800 50  0001 C CNN
+F 2 "Resistor_SMD:R_0603_1608Metric_Pad1.05x0.95mm_HandSolder" V 6180 4800 50  0001 C CNN
 F 3 "~" H 6250 4800 50  0001 C CNN
 	1    6250 4800
@@
 F 0 "R5" H 7970 2796 50  0000 L CNN
 F 1 "10k" H 7970 2705 50  0000 L CNN
-F 2 "Resistor_SMD:R_0805_2012Metric_Pad1.15x1.40mm_HandSolder" V 7830 2750 50  0001 C CNN
+F 2 "Resistor_SMD:R_0603_1608Metric_Pad1.05x0.95mm_HandSolder" V 7830 2750 50  0001 C CNN
 F 3 "~" H 7900 2750 50  0001 C CNN
 	1    7900 2750
@@
 F 0 "R6" H 7970 3446 50  0000 L CNN
 F 1 "10k" H 7970 3355 50  0000 L CNN
-F 2 "Resistor_SMD:R_0805_2012Metric_Pad1.15x1.40mm_HandSolder" V 7830 3400 50  0001 C CNN
+F 2 "Resistor_SMD:R_0603_1608Metric_Pad1.05x0.95mm_HandSolder" V 7830 3400 50  0001 C CNN
 F 3 "~" H 7900 3400 50  0001 C CNN
 	1    7900 3400
@@
 F 0 "R7" H 7970 4146 50  0000 L CNN
 F 1 "10k" H 7970 4055 50  0000 L CNN
-F 2 "Resistor_SMD:R_0805_2012Metric_Pad1.15x1.40mm_HandSolder" V 7830 4100 50  0001 C CNN
+F 2 "Resistor_SMD:R_0603_1608Metric_Pad1.05x0.95mm_HandSolder" V 7830 4100 50  0001 C CNN
 F 3 "~" H 7900 4100 50  0001 C CNN
 	1    7900 4100
@@
 F 0 "R8" H 7970 4846 50  0000 L CNN
 F 1 "10k" H 7970 4755 50  0000 L CNN
-F 2 "Resistor_SMD:R_0805_2012Metric_Pad1.15x1.40mm_HandSolder" V 7830 4800 50  0001 C CNN
+F 2 "Resistor_SMD:R_0603_1608Metric_Pad1.05x0.95mm_HandSolder" V 7830 4800 50  0001 C CNN
 F 3 "~" H 7900 4800 50  0001 C CNN
 	1    7900 4800
@@
 F 0 "R9" H 9720 2646 50  0000 L CNN
 F 1 "10k" H 9720 2555 50  0000 L CNN
-F 2 "Resistor_SMD:R_0805_2012Metric_Pad1.15x1.40mm_HandSolder" V 9580 2600 50  0001 C CNN
+F 2 "Resistor_SMD:R_0603_1608Metric_Pad1.05x0.95mm_HandSolder" V 9580 2600 50  0001 C CNN
 F 3 "~" H 9650 2600 50  0001 C CNN
 	1    9650 2600
@@
 F 0 "R10" H 9720 3296 50  0000 L CNN
 F 1 "10k" H 9720 3205 50  0000 L CNN
-F 2 "Resistor_SMD:R_0805_2012Metric_Pad1.15x1.40mm_HandSolder" V 9580 3250 50  0001 C CNN
+F 2 "Resistor_SMD:R_0603_1608Metric_Pad1.05x0.95mm_HandSolder" V 9580 3250 50  0001 C CNN
 F 3 "~" H 9650 3250 50  0001 C CNN
 	1    9650 3250
@@
 F 0 "D1" H 10093 3945 50  0000 C CNN
 F 1 "LED" H 10093 4036 50  0000 C CNN
-F 2 "LED_SMD:LED_0805_2012Metric_Pad1.15x1.40mm_HandSolder" H 10100 4200 50  0001 C CNN
+F 2 "LED_SMD:LED_0603_1608Metric_Pad1.05x0.95mm_HandSolder" H 10100 4200 50  0001 C CNN
 F 3 "~" H 10100 4200 50  0001 C CNN
 	1    10100 4200
@@
 F 0 "R11" V 9443 4200 50  0000 C CNN
 F 1 "330" V 9534 4200 50  0000 C CNN
-F 2 "Resistor_SMD:R_0805_2012Metric_Pad1.15x1.40mm_HandSolder" V 9580 4200 50  0001 C CNN
+F 2 "Resistor_SMD:R_0603_1608Metric_Pad1.05x0.95mm_HandSolder" V 9580 4200 50  0001 C CNN
 F 3 "~" H 9650 4200 50  0001 C CNN
 	1    9650 4200
