File: monitor-board/monitor-board.kicad_pcb (KiCad board)
At the start: 2 copper layers, 55.9 x 53.3 mm, 26 parts, among them J1 Conn_01x06, SW1 SW_IO12, SW2 SW_IO13, SW3 SW_IO14, SW4 SW_IO15, SW5 SW_IO32, SW6 SW_IO33, SW7 SW_IO34, SW8 SW_IO35, U1 ESP32-WROOM-32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

Commit message: update silkscreen
Other:
- board text added: "Chris Johnston 10/30/2019 rev 0 github.com/Chris-Johnston"
- board text added: "https://github.com/Chris-Johnston/door-monitor/"
- board text removed: "Chris Johnston 10/30/2019 github.com/Chris-Johnston"
Changed lines of the file:
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@@
   (general
     (thickness 1.6)
-    (drawings 14)
+    (drawings 15)
     (tracks 225)
     (zones 0)
@@
     (0 F.Cu signal hide)
     (31 B.Cu signal hide)
-    (33 F.Adhes user hide)
-    (35 F.Paste user hide)
+    (33 F.Adhes user)
+    (35 F.Paste user)
     (36 B.SilkS user)
     (37 F.SilkS user)
     (39 F.Mask user)
-    (40 Dwgs.User user hide)
-    (41 Cmts.User user hide)
-    (42 Eco1.User user hide)
-    (43 Eco2.User user hide)
+    (40 Dwgs.User user)
+    (41 Cmts.User user)
+    (42 Eco1.User user)
+    (43 Eco2.User user)
     (44 Edge.Cuts user)
-    (45 Margin user hide)
-    (46 B.CrtYd user hide)
-    (47 F.CrtYd user hide)
-    (49 F.Fab user hide)
+    (45 Margin user)
+    (46 B.CrtYd user)
+    (47 F.CrtYd user)
+    (49 F.Fab user)
   )
   (setup
@@
     )
   )
+  (gr_text https://github.com/Chris-Johnston/door-monitor/ (at 52.07 35.56) (layer B.SilkS)
+    (effects (font (size 1 0.8) (thickness 0.2)) (justify mirror))
+  )
   (gr_text "NOT A BOMB" (at 65.913 33.401 90) (layer F.SilkS)
     (effects (font (size 1 1) (thickness 0.15)))
@@
     (effects (font (size 0.5 0.5) (thickness 0.125)))
   )
-  (gr_text "Chris Johnston 10/30/2019\ngithub.com/Chris-Johnston" (at 48.26 28.448) (layer F.SilkS)
-    (effects (font (size 1 1) (thickness 0.15)))
+  (gr_text "Chris Johnston 10/30/2019 rev 0\ngithub.com/Chris-Johnston\n" (at 38.1 28.448) (layer F.SilkS)
+    (effects (font (size 1 1) (thickness 0.15)) (justify left))
   )
   (gr_text "if you can read\nthis, the board hasn't\nbeen assembled yet" (at 53.086 52.832) (layer F.SilkS)
